File: RF Project/Tx-Rx.sch (KiCad schematic (older format))
At the start: 26 parts, among them J1 CONN_Right, J2 CONN_Left, U1 CC2500RGPR, U2 U.FL_male

Commit message: Add files via upload
Parts:
- C14, C16, C17: value 220μF -> 220pF
Changed lines of the file:
@@
 LIBS:contrib
 LIBS:valves
-LIBS:cc2500rgpr
 LIBS:Tx-Rx-cache
 EELAYER 25 0
@@
 P 9550 1750
 F 0 "C14" H 9575 1850 50  0000 L CNN
-F 1 "220μF" H 9575 1650 50  0000 L CNN
+F 1 "220pF" H 9575 1650 50  0000 L CNN
 F 2 "Capacitors_SMD:C_0402" H 9588 1600 50  0001 C CNN
 F 3 "" H 9550 1750 50  0001 C CNN
@@
 P 10300 1750
 F 0 "C16" H 10325 1850 50  0000 L CNN
-F 1 "220μF" H 10325 1650 50  0000 L CNN
+F 1 "220pF" H 10325 1650 50  0000 L CNN
 F 2 "Capacitors_SMD:C_0402" H 10338 1600 50  0001 C CNN
 F 3 "" H 10300 1750 50  0001 C CNN
@@
 P 10550 2650
 F 0 "C17" H 10575 2750 50  0000 L CNN
-F 1 "220μF" H 10575 2550 50  0000 L CNN
+F 1 "220pF" H 10575 2550 50  0000 L CNN
 F 2 "Capacitors_SMD:C_0402" H 10588 2500 50  0001 C CNN
 F 3 "" H 10550 2650 50  0001 C CNN
