File: RF Project/GPS.sch (KiCad schematic (older format))
At the start: 10 parts, among them U11 Venus634SMD, U3 U.FL_male

Commit message: revision component placement, coupling caps added
Parts:
- added C21, C22, C23: 1uF, Capacitors_SMD:C_0402, symbol C
Connections:
- net RF_GND is gone; now on net GNDREF: C19.1, U11.21 (GNDRF), U11.22 (GNDRF), U11.24 (GNDRF), U11.25 (GNDRF), U11.27 (GNDRF), U11.28 (GNDRF), U11.29 (GNDRF), U11.31 (GNDRF), U11.33 (GNDRF), U3.1 (GND), U3.2 (GND)
- net GNDREF: now also C21.2, C22.2, C23.2
- net VCC: now also C21.1, C22.1, C23.1
- net RFIN: no longer names the net of L4.2, U11.32 (RFIN), U3.3 (DATA)
Other:
- note added: "Cap used for low power jumper\n"
- note added: "Coupling Caps"
- note removed: "CONNECT TO NAV????\n"
- note removed: "CORRECT GPIO? Cap used for low power jumper\n"
Changed lines of the file:
@@
 $EndComp
 $Comp
-L VCC #PWR021
-U 1 1 5B56D218
-P 6750 2500
-F 0 "#PWR021" H 6750 2350 50  0001 C CNN
-F 1 "VCC" H 6750 2650 50  0000 C CNN
-F 2 "" H 6750 2500 50  0001 C CNN
-F 3 "" H 6750 2500 50  0001 C CNN
-	1    6750 2500
-	1    0    0    -1
-$EndComp
-$Comp
-L GNDREF #PWR022
+L GNDREF #PWR021
 U 1 1 5B56D409
 P 7125 4250
-F 0 "#PWR022" H 7125 4000 50  0001 C CNN
+F 0 "#PWR021" H 7125 4000 50  0001 C CNN
 F 1 "GNDREF" H 7125 4100 50  0000 C CNN
 F 2 "" H 7125 4250 50  0001 C CNN
@@
 $EndComp
 $Comp
-L GNDREF #PWR023
+L GNDREF #PWR022
 U 1 1 5B56D55E
 P 7450 4250
-F 0 "#PWR023" H 7450 4000 50  0001 C CNN
+F 0 "#PWR022" H 7450 4000 50  0001 C CNN
 F 1 "GNDREF" H 7450 4100 50  0000 C CNN
 F 2 "" H 7450 4250 50  0001 C CNN
@@
 $EndComp
 $Comp
-L GNDREF #PWR024
+L GNDREF #PWR023
 U 1 1 5B56D575
 P 7800 4250
-F 0 "#PWR024" H 7800 4000 50  0001 C CNN
+F 0 "#PWR023" H 7800 4000 50  0001 C CNN
 F 1 "GNDREF" H 7800 4100 50  0000 C CNN
 F 2 "" H 7800 4250 50  0001 C CNN
@@
 	1    7800 2650
 	1    0    0    -1
-$EndComp
-$Comp
-L VCC #PWR025
-U 1 1 5B56D608
-P 7800 2350
-F 0 "#PWR025" H 7800 2200 50  0001 C CNN
-F 1 "VCC" H 7800 2500 50  0000 C CNN
-F 2 "" H 7800 2350 50  0001 C CNN
-F 3 "" H 7800 2350 50  0001 C CNN
-	1    7800 2350
-	1    0    0    -1
-$EndComp
-$Comp
-L U.FL_male U3
-U 1 1 5B56DE12
-P 4050 3100
-F 0 "U3" H 4050 2600 60  0000 C CNN
-F 1 "U.FL_male" H 4100 3450 60  0000 C CNN
-F 2 "RF_Transciever:u.fl_male" H 4050 3100 60  0001 C CNN
-F 3 "" H 4050 3100 60  0001 C CNN
-	1    4050 3100
-	-1   0    0    1
 $EndComp
 $Comp
@@
 $EndComp
 $Comp
-L VCC #PWR026
+L VCC #PWR025
 U 1 1 5B56E2CF
 P 3200 2625
-F 0 "#PWR026" H 3200 2475 50  0001 C CNN
+F 0 "#PWR025" H 3200 2475 50  0001 C CNN
 F 1 "VCC" H 3200 2775 50  0000 C CNN
 F 2 "" H 3200 2625 50  0001 C CNN
@@
 F 3 "" H 6625 5600 50  0001 C CNN
 	1    6625 5600
-	1    0    0    -1
-$EndComp
-$Comp
-L VCC #PWR027
-U 1 1 5B56E543
-P 7300 5475
-F 0 "#PWR027" H 7300 5325 50  0001 C CNN
-F 1 "VCC" H 7300 5625 50  0000 C CNN
-F 2 "" H 7300 5475 50  0001 C CNN
-F 3 "" H 7300 5475 50  0001 C CNN
-	1    7300 5475
 	1    0    0    -1
 $EndComp
@@
 $EndComp
 $Comp
-L GNDREF #PWR028
+L GNDREF #PWR026
 U 1 1 5B56EFB5
 P 2775 1500
-F 0 "#PWR028" H 2775 1250 50  0001 C CNN
+F 0 "#PWR026" H 2775 1250 50  0001 C CNN
 F 1 "GNDREF" H 2775 1350 50  0000 C CNN
 F 2 "" H 2775 1500 50  0001 C CNN
@@
 Text GLabel 6700 3875 2    60   Input ~ 0
 GPIO24
-Text GLabel 2025 775  0    60   Input ~ 0
+Text GLabel 2125 775  0    60   Input ~ 0
 TX
-Text HLabel 2125 775  2    60   Input ~ 0
+Text HLabel 2225 775  2    60   Input ~ 0
 TX
-Text GLabel 2025 925  0    60   Input ~ 0
+Text GLabel 2125 925  0    60   Input ~ 0
 RX
-Text HLabel 2125 925  2    60   Input ~ 0
+Text HLabel 2225 925  2    60   Input ~ 0
 RX
 Text GLabel 5100 4875 3    60   Input ~ 0
 RF_GND
-Text Label 4850 2750 0    60   ~ 0
-RFIN
 Text GLabel 4500 3250 3    60   Input ~ 0
 RF_GND
 Text GLabel 3600 3250 3    60   Input ~ 0
 RF_GND
-Wire Wire Line
-	6575 2750 6750 2750
-Wire Wire Line
-	6750 2500 6750 2875
-Wire Wire Line
-	6750 2875 6575 2875
-Connection ~ 6750 2750
 Wire Wire Line
 	6700 4750 6575 4750
@@
 	1275 1250 1275 1175
 Wire Wire Line
-	3725 2750 5225 2750
-Connection ~ 4050 2750
-Wire Wire Line
 	3200 2750 3425 2750
 Wire Wire Line
@@
 Connection ~ 3200 2750
 Wire Wire Line
-	6775 5600 7300 5600
-Wire Wire Line
-	7300 5600 7300 5475
-Wire Wire Line
 	6275 5600 6475 5600
 Wire Wire Line
@@
 	5100 3750 5225 3750
 Wire Wire Line
-	2025 775  2125 775
-Wire Wire Line
-	2125 925  2025 925
+	2125 775  2225 775
+Wire Wire Line
+	2225 925  2125 925
 Connection ~ 5100 4750
 Wire Wire Line
@@
 Wire Wire Line
 	3200 3175 3200 3250
-Text Label 6900 3125 0    60   ~ 0
+Text Label 7100 3125 0    60   ~ 0
 BTSEL
-Text Label 6900 3000 0    60   ~ 0
+Text Label 7100 3000 0    60   ~ 0
 RSTN
 Text GLabel 5750 5600 0    60   Input ~ 0
 NAV
-Text Notes 5300 5825 0    60   ~ 0
-CONNECT TO NAV????\n
-Text Notes 2925 875  0    60   ~ 0
-CORRECT GPIO? Cap used for low power jumper\n
+Text Notes 2075 1800 0    60   ~ 0
+Cap used for low power jumper\n
 $Comp
 L C lw_pwr1
@@
 Wire Wire Line
 	2775 1050 2775 1000
+Text GLabel 1600 1275 3    60   Input ~ 0
+RF_GND
+Text HLabel 1600 1175 1    60   Input ~ 0
+PWR_GND
+Wire Wire Line
+	1600 1275 1600 1175
+Wire Notes Line
+	4200 625  4200 1950
+Wire Notes Line
+	4200 1950 7575 1950
+Wire Notes Line
+	7575 1950 7575 625
+Wire Notes Line
+	7575 625  4200 625
+Text Notes 5375 2100 0    60   ~ 0
+Coupling Caps
+Wire Wire Line
+	3725 2750 5225 2750
+Wire Wire Line
+	5125 1500 5125 900
+$Comp
+L VCC #PWR027
+U 1 1 5BA2F261
+P 5125 900
+F 0 "#PWR027" H 5125 750 50  0001 C CNN
+F 1 "VCC" H 5125 1050 50  0000 C CNN
+F 2 "" H 5125 900 50  0001 C CNN
+F 3 "" H 5125 900 50  0001 C CNN
+	1    5125 900
+	1    0    0    -1
+$EndComp
+Connection ~ 5125 1150
+$Comp
+L C C21
+U 1 1 5BA2F476
+P 5425 1300
+F 0 "C21" H 5450 1400 50  0000 L CNN
+F 1 "1uF" H 5450 1200 50  0000 L CNN
+F 2 "Capacitors_SMD:C_0402" H 5463 1150 50  0001 C CNN
+F 3 "" H 5425 1300 50  0001 C CNN
+	1    5425 1300
+	1    0    0    -1
+$EndComp
+Wire Wire Line
+	5425 1450 5425 1500
+$Comp
+L GNDREF #PWR028
+U 1 1 5BA2F7E8
+P 5425 1500
+F 0 "#PWR028" H 5425 1250 50  0001 C CNN
+F 1 "GNDREF" H 5425 1350 50  0000 C CNN
+F 2 "" H 5425 1500 50  0001 C CNN
+F 3 "" H 5425 1500 50  0001 C CNN
+	1    5425 1500
+	1    0    0    -1
+$EndComp
+Wire Wire Line
+	5425 1150 5125 1150
+Connection ~ 4050 2750
+Wire Wire Line
+	5800 1500 5800 900
+$Comp
+L VCC #PWR029
+U 1 1 5BA314F5
+P 5800 900
+F 0 "#PWR029" H 5800 750 50  0001 C CNN
+F 1 "VCC" H 5800 1050 50  0000 C CNN
+F 2 "" H 5800 900 50  0001 C CNN
+F 3 "" H 5800 900 50  0001 C CNN
+	1    5800 900
+	1    0    0    -1
+$EndComp
+Connection ~ 5800 1150
+$Comp
+L C C22
+U 1 1 5BA314FC
+P 6100 1300
+F 0 "C22" H 6125 1400 50  0000 L CNN
+F 1 "1uF" H 6125 1200 50  0000 L CNN
+F 2 "Capacitors_SMD:C_0402" H 6138 1150 50  0001 C CNN
+F 3 "" H 6100 1300 50  0001 C CNN
+	1    6100 1300
+	1    0    0    -1
+$EndComp
+Wire Wire Line
+	6100 1450 6100 1500
+$Comp
+L GNDREF #PWR030
+U 1 1 5BA31503
+P 6100 1500
+F 0 "#PWR030" H 6100 1250 50  0001 C CNN
+F 1 "GNDREF" H 6100 1350 50  0000 C CNN
+F 2 "" H 6100 1500 50  0001 C CNN
+F 3 "" H 6100 1500 50  0001 C CNN
+	1    6100 1500
+	1    0    0    -1
+$EndComp
+Wire Wire Line
+	6100 1150 5800 1150
+Wire Wire Line
+	6575 2750 6700 2750
+Wire Wire Line
+	6575 2875 6700 2875
+Text GLabel 6700 2750 2    60   Input ~ 0
+VCCCPL
+Text GLabel 6700 2875 2    60   Input ~ 0
+REGEN
+Wire Wire Line
+	6425 1500 6425 900
+$Comp
+L VCC #PWR031
+U 1 1 5BA31DC5
+P 6425 900
+F 0 "#PWR031" H 6425 750 50  0001 C CNN
+F 1 "VCC" H 6425 1050 50  0000 C CNN
+F 2 "" H 6425 900 50  0001 C CNN
+F 3 "" H 6425 900 50  0001 C CNN
+	1    6425 900
+	1    0    0    -1
+$EndComp
+Connection ~ 6425 1150
+$Comp
+L C C23
+U 1 1 5BA31DCC
+P 6725 1300
+F 0 "C23" H 6750 1400 50  0000 L CNN
+F 1 "1uF" H 6750 1200 50  0000 L CNN
+F 2 "Capacitors_SMD:C_0402" H 6763 1150 50  0001 C CNN
+F 3 "" H 6725 1300 50  0001 C CNN
+	1    6725 1300
+	1    0    0    -1
+$EndComp
+Wire Wire Line
+	6725 1450 6725 1500
+$Comp
+L GNDREF #PWR032
+U 1 1 5BA31DD3
+P 6725 1500
+F 0 "#PWR032" H 6725 1250 50  0001 C CNN
+F 1 "GNDREF" H 6725 1350 50  0000 C CNN
+F 2 "" H 6725 1500 50  0001 C CNN
+F 3 "" H 6725 1500 50  0001 C CNN
+	1    6725 1500
+	1    0    0    -1
+$EndComp
+Wire Wire Line
+	6725 1150 6425 1150
+Text GLabel 6425 1500 3    60   Input ~ 0
+REGEN
+Text GLabel 5800 1500 3    60   Input ~ 0
+VCCCPL
+$Comp
+L U.FL_male U3
+U 1 1 5B56DE12
+P 4050 3100
+F 0 "U3" H 4050 2600 60  0000 C CNN
+F 1 "U.FL_male" H 4100 3450 60  0000 C CNN
+F 2 "RF_Transciever:u.fl_male" H 4050 3100 60  0001 C CNN
+F 3 "" H 4050 3100 60  0001 C CNN
+	1    4050 3100
+	-1   0    0    1
+$EndComp
+Wire Wire Line
+	6775 5600 7000 5600
+Text GLabel 7000 5600 2    60   Input ~ 0
+LEDVCC
+Text GLabel 5125 1500 3    60   Input ~ 0
+LEDVCC
+$Comp
+L VCC #PWR024
+U 1 1 5B56D608
+P 7800 2350
+F 0 "#PWR024" H 7800 2200 50  0001 C CNN
+F 1 "VCC" H 7800 2500 50  0000 C CNN
+F 2 "" H 7800 2350 50  0001 C CNN
+F 3 "" H 7800 2350 50  0001 C CNN
+	1    7800 2350
+	1    0    0    -1
+$EndComp
 $EndSCHEMATC
